Commit message: correct collision urdf

File: humanoid_description/urdf/humanoid.urdf.xacro (robot description, xacro)
@@ -27,5 +27,5 @@
     </visual>
      <collision>
-      <origin rpy="1.57 0  1.57" xyz="0.85 -.42 1.4"/>
+      <origin rpy="1.57 0  1.57" xyz="0.85 -.44 1.4"/>
       <geometry>
          <mesh filename="package://humanoid_description/urdf/torso.stl" scale="0.001 0.001 0.001"/>

Commit message: updated stl from vention with plate for PTU

File: humanoid_description/urdf/humanoid.urdf.xacro (robot description, xacro)
@@ -23,5 +23,5 @@
       <origin rpy="1.57 0  1.57" xyz="0.85 -.44 1.4"/>
       <geometry>
-         <mesh filename="package://humanoid_description/urdf/torso.stl" scale="0.001 0.001 0.001"/>
+         <mesh filename="package://humanoid_description/meshes/VentionAssembly_159315_v38.stl" scale="0.001 0.001 0.001"/>
       </geometry>
     </visual>
@@ -29,5 +29,5 @@
       <origin rpy="1.57 0  1.57" xyz="0.85 -.44 1.4"/>
       <geometry>
-         <mesh filename="package://humanoid_description/urdf/torso.stl" scale="0.001 0.001 0.001"/>
+         <mesh filename="package://humanoid_description/meshes/VentionAssembly_159315_v38.stl" scale="0.001 0.001 0.001"/>
       </geometry>
     </collision>

Commit message: add ptu to description

File: humanoid_description/urdf/humanoid.urdf.xacro (robot description, xacro)
@@ -8,4 +8,5 @@
   <!--  Arguments for the iiwa7 macro  -->
   <xacro:arg name="hardware_interface" default="PositionJointInterface"/>
+  <!-- Define world -->
   <link name="world">
     <origin xyz ="0.0 0.0 0.0" rpy="0 0 0"/>
@@ -19,4 +20,5 @@
     <origin xyz ="0.0 0.0 0.0" rpy="0 0 0"/>
   </joint>
+  <!-- Define torso from Vention -->
   <link name="torso">
     <visual>
@@ -41,3 +43,12 @@
     <origin xyz="0.15 -0.33 1.35" rpy="0 1.57 0"/>
   </xacro:iiwa7>
+ <!-- Include and invoke the macro which creates a D46 PTU -->
+  <xacro:include filename="$(find flir_ptu_description)/urdf/d46.urdf.xacro" />
+  <xacro:ptu_d46 name="ptu" />
+  <!-- Create a fixed joint to connect the PTU to the rest of the robot -->
+  <joint name="torso_to_ptu_base" type="fixed">
+    <parent link="torso"/>
+    <child link="ptu_base_link"/>
+    <origin xyz="0.1 -0.01 1.54"/>
+  </joint>
 </robot>

Commit message: first pass at PTU to SC calib

File: humanoid_description/urdf/humanoid.urdf.xacro (robot description, xacro)
@@ -52,3 +52,12 @@
     <origin xyz="0.1 -0.01 1.54"/>
   </joint>
+  <!-- PTU to SC -->
+  <joint name="ptu_to_sc" type="fixed">
+    <parent link="ptu_mount_link"/>
+    <child link="sc_map"/>
+    <origin xyz="0.0 0.0 0" rpy="-1.570 0 -1.57"/>
+  </joint>
+  <link name="sc_map">
+    <origin xyz ="0.0 0.0 0" rpy="0 0 0"/>
+  </link>
 </robot>

Commit message: very precise table positioning

File: humanoid_description/urdf/humanoid.urdf.xacro (robot description, xacro)
@@ -61,3 +61,24 @@
     <origin xyz ="0.0 0.0 0" rpy="0 0 0"/>
   </link>
+  <!-- APPROXIMATE TABLE HEIGHT -->
+  <joint name="world_to_table" type="fixed">
+    <parent link="world"/>
+    <child link="table"/>
+    <origin xyz="0.0 0.0 0.75087592"/>
+  </joint>
+  <link name="table">
+    <visual>
+      <geometry>
+         <box size="5.0 5.0 0.01"/>
+      </geometry>
+      <material name="grey">
+        <color rgba="0.5 0.5 0.5 1"/>
+      </material>
+    </visual>
+     <collision>
+      <geometry>
+         <box size="5.0 5.0 0.01"/>
+      </geometry>
+    </collision>
+  </link>
 </robot>

Commit message: SDH, FT in URDF. WIP FT DIMENSIONS

File: humanoid_description/urdf/humanoid.urdf.xacro (robot description, xacro)
@@ -8,4 +8,8 @@
   <!--  Arguments for the iiwa7 macro  -->
   <xacro:arg name="hardware_interface" default="PositionJointInterface"/>
+  <!--  Edit  -->
+  <!--Import the schunk sdh macro -->
+  <xacro:include filename="$(find schunk_description)/urdf/sdh/sdh.urdf.xacro"/>
+  <!--  Edit  -->
   <!-- Define world -->
   <link name="world">
@@ -43,4 +47,42 @@
     <origin xyz="0.15 -0.33 1.35" rpy="0 1.57 0"/>
   </xacro:iiwa7>
+  <!--  Edit  -->
+<!--   <link name="ft_sensor_right">
+    <visual>
+      <geometry>
+         <box size="0.3 0.3 0.01"/>
+      </geometry>
+      <material name="yellow">
+        <color rgba="0.5 0.0 0.5 1"/>
+      </material>
+    </visual>
+     <collision>
+      <geometry>
+         <box size="0.3 0.3 0.01"/>
+      </geometry>
+    </collision>
+  <joint name="iiwa_right_to_ft_sensor_right" type="fixed">
+    <parent link="iiwa_right_link_ee"/>
+    <child link="ft_sensor_right"/>
+    <origin xyz="0.0 0.0 0.01"/>
+  </joint>
+  </link> -->
+  <!--Here we insert the (right) Schunk SDH2 in the scene -->
+  <xacro:schunk_sdh name="schunk_right" parent="iiwa_right_link_ee">
+    <origin xyz="0 0 0.01" rpy="0 0 0"/>
+  </xacro:schunk_sdh>
+  <!-- define SchunkRight_ee_link such that iiwa_ros finds the tool frame -->
+  <joint name="right_ee_fixed" type="fixed">
+    <parent link="iiwa_right_link_ee" />
+    <child link="SchunkRight_link_ee"/>
+    <origin xyz="0 0 0.134"/>
+  </joint>
+  <link name="SchunkRight_link_ee"/>
+<!--   <joint name="iiwa_right_to_schunk_right" type="fixed">
+    <parent link="iiwa_right_joint_ee"/>
+    <child link="schunk_right"/>
+    <origin xyz="0 0 0.1"/>
+  </joint> -->
+  <!--  Edit  -->
  <!-- Include and invoke the macro which creates a D46 PTU -->
   <xacro:include filename="$(find flir_ptu_description)/urdf/d46.urdf.xacro" />

Commit message: urdf modeling adapter & wrist FT properly. adjusting structure core position as well

File: humanoid_description/urdf/humanoid.urdf.xacro (robot description, xacro)
@@ -47,28 +47,27 @@
     <origin xyz="0.15 -0.33 1.35" rpy="0 1.57 0"/>
   </xacro:iiwa7>
-  <!--  Edit  -->
-<!--   <link name="ft_sensor_right">
+  <joint name="iiwa_right_to_ft_sensor_right" type="fixed">
+    <parent link="iiwa_right_link_ee"/>
+    <child link="ft_sensor_right"/>
+    <origin xyz="0.0 0.0 0.0635"/>
+  </joint>
+  <link name="ft_sensor_right">
     <visual>
       <geometry>
-         <box size="0.3 0.3 0.01"/>
+         <cylinder radius="0.0508" length="0.127"/>
       </geometry>
       <material name="yellow">
-        <color rgba="0.5 0.0 0.5 1"/>
+        <color rgba="0.75 0.75 0.75 1"/>
       </material>
     </visual>
      <collision>
       <geometry>
-         <box size="0.3 0.3 0.01"/>
+         <cylinder radius="0.0508" length="0.127"/>
       </geometry>
     </collision>
-  <joint name="iiwa_right_to_ft_sensor_right" type="fixed">
-    <parent link="iiwa_right_link_ee"/>
-    <child link="ft_sensor_right"/>
-    <origin xyz="0.0 0.0 0.01"/>
-  </joint>
-  </link> -->
+  </link>
   <!--Here we insert the (right) Schunk SDH2 in the scene -->
-  <xacro:schunk_sdh name="schunk_right" parent="iiwa_right_link_ee">
-    <origin xyz="0 0 0.01" rpy="0 0 0"/>
+  <xacro:schunk_sdh name="schunk_right" parent="ft_sensor_right">
+    <origin xyz="0 0 0.0635" rpy="0 0 -1.8"/>
   </xacro:schunk_sdh>
   <!-- define SchunkRight_ee_link such that iiwa_ros finds the tool frame -->
@@ -92,5 +91,5 @@
     <parent link="torso"/>
     <child link="ptu_base_link"/>
-    <origin xyz="0.1 -0.01 1.54"/>
+    <origin xyz="0.11 -0.01 1.54"/>
   </joint>
   <!-- PTU to SC -->
@@ -98,5 +97,6 @@
     <parent link="ptu_mount_link"/>
     <child link="sc_map"/>
-    <origin xyz="0.0 0.0 0" rpy="-1.570 0 -1.57"/>
+    <!-- <origin xyz="0.0206375 0.0 0.01905" rpy="-1.570 0 -1.57"/> -->
+    <origin xyz="0.01 0.0 0.0" rpy="-1.570 0 -1.57"/>
   </joint>
   <link name="sc_map">
@@ -104,5 +104,5 @@
   </link>
   <!-- APPROXIMATE TABLE HEIGHT -->
-  <joint name="world_to_table" type="fixed">
+  <!-- <joint name="world_to_table" type="fixed">
     <parent link="world"/>
     <child link="table"/>
@@ -123,4 +123,4 @@
       </geometry>
     </collision>
-  </link>
+  </link> -->
 </robot>

Commit message: motor skills submod; moveit redo after fixing FT sensor, disable adjacent collisions now. gripper_joint_traj_test now lives in motor_skills/ros

File: humanoid_description/urdf/humanoid.urdf.xacro (robot description, xacro)
@@ -55,5 +55,5 @@
     <visual>
       <geometry>
-         <cylinder radius="0.0508" length="0.127"/>
+         <cylinder radius="0.0508" length="0.125"/>
       </geometry>
       <material name="yellow">
@@ -63,5 +63,5 @@
      <collision>
       <geometry>
-         <cylinder radius="0.0508" length="0.127"/>
+         <cylinder radius="0.0508" length="0.125"/>
       </geometry>
     </collision>

Commit message: object modeled for motion planning around it

File: humanoid_description/urdf/humanoid.urdf.xacro (robot description, xacro)
@@ -103,4 +103,44 @@
     <origin xyz ="0.0 0.0 0" rpy="0 0 0"/>
   </link>
+  <joint name="world_to_obj" type="fixed">
+    <parent link="world"/>
+    <child link="obj"/>
+    <origin xyz="1.55 0.65 1.2" rpy="0 0 0.65"/>
+  </joint>
+  <link name="obj">
+    <visual>
+      <geometry>
+        <box size="1.0 1.5 1"/>
+      </geometry>
+      <material name="grey">
+        <color rgba="0.5 0.5 0.5 0.5"/>
+      </material>
+    </visual>
+     <collision>
+      <geometry>
+        <box size="1.0 1.5 1"/>
+      </geometry>
+    </collision>
+  </link>
+  <joint name="obj_to_obj2" type="fixed">
+    <parent link="obj"/>
+    <child link="obj2"/>
+    <origin xyz="-0.3 -0.55 0" rpy="0 0 0.0"/>
+  </joint>
+  <link name="obj2">
+    <visual>
+      <geometry>
+         <box size="1.0 0.3 1"/>
+      </geometry>
+      <material name="grey">
+        <color rgba="0.5 0.5 0.5 0.5"/>
+      </material>
+    </visual>
+     <collision>
+      <geometry>
+         <box size="1.0 0.3 1"/>
+      </geometry>
+    </collision>
+  </link>
   <!-- APPROXIMATE TABLE HEIGHT -->
   <!-- <joint name="world_to_table" type="fixed">
